File: Adaptor/Adaptor.brd (EAGLE design)
At the start: 120 x 120 mm, 10 parts

Commit message: cleanm up.
Parts:
- removed C1: 100n, Wurth_Elektronik_Passive_Capacitors_rev19a:WCAP-CSGP_0402
- removed R1, R2: 4k7, Resistor_smaller_fliegl:WCAP-CSRF_0402
- removed U2: (no value), BTS7030-2EPA:SOP65P600X115-15N-V
- GND, IN0, IN1, OUT0, OUT1, VS: value 9774100982 -> M4 x 10mm; device Wurth_Assembly_WA-SMST:WA-SMST_9774100982 -> Wurth_Assembly_WA-SMSI:WA-SMSI_9774100482
Connections:
- removed net GND: C1.2, GND.1, U2.1
- removed net IN0: IN0.1, R2.1
- removed net IN1: IN1.1, R1.1
- removed net N$16: R2.2, U2.2
- removed net N$18: R1.2, U2.6
- removed net OUT0: OUT0.1, U2.12, U2.13, U2.14
- removed net OUT1: OUT1.1, U2.10, U2.8, U2.9
- removed net VCC: C1.1, U2.15, VS.1
Routing:
- net GND: track 61.7 -> 0.00 mm
- net OUT1: track 44.6 -> 0.00 mm
- net OUT0: track 44.6 -> 0.00 mm
- net IN1: track 40.7 -> 0.00 mm
- net IN0: track 40.7 -> 0.00 mm
- net N$18: track 3.15 -> 0.00 mm
- net N$16: track 3.15 -> 0.00 mm
- removed copper zone on layer 1, net OUT0
- removed copper zone on layer 1, net OUT1
- removed copper zone on layer 1, net VCC
- removed copper zone on layer 16, net VCC

Commit message: finish !
Parts:
- removed GND, IN0, IN1, OUT0, OUT1, VS: M4 x 10mm, Wurth_Assembly_WA-SMSI:WA-SMSI_9774100482
- added 1, 1', 2, 2', 3, 3', 4, 4', 5, 6: M4 x 10mm, Wurth_Assembly_WA-SMSI:WA-SMSI_9774100482
- added J1: 638207222006, Wurth_Connectors_WR-FAST:638207222006
- added J2: 638207222004, Wurth_Connectors_WR-FAST:638207222004
Connections:
- new net N$1: 1.1, J1.1, J1.A1
- new net N$10: 3'.1, J2.3, J2.A3
- new net N$2: 2.1, J1.2, J1.A2
- new net N$3: 3.1, J1.3, J1.A3
- new net N$4: 4.1, J1.4, J1.A4
- new net N$5: 5.1, J1.5, J1.A5
- new net N$6: 6.1, J1.6, J1.A6
- new net N$7: 1'.1, J2.1, J2.A1
- new net N$8: 2'.1, J2.2, J2.A2
- new net N$9: 4'.1, J2.4, J2.A4
Routing:
- net N$5: track 0.00 -> 48.4 mm
- net N$2: track 0.00 -> 48.4 mm
- net N$10: track 0.00 -> 46.3 mm
- net N$1: track 0.00 -> 46.3 mm
- net N$8: track 0.00 -> 46.3 mm
- net N$6: track 0.00 -> 46.3 mm
- net N$9: track 0.00 -> 44.2 mm
- net N$7: track 0.00 -> 44.2 mm
- net N$4: track 0.00 -> 44.2 mm
- net N$3: track 0.00 -> 44.2 mm
